File: _autosave-high_power_dc_load_control_unit.kicad_sch (KiCad schematic)
At the start: 53 parts, among them IC1 STPS60L45CW, IC3 LT8711EFE#TRPBF, J4 XT60-M, J5 XT60-M, Q1 RS6P100BHTB1, Q2 PMOS, Q4 NMOS, U1 UCC5350MCD, U2 LTC3525ESC6-5-TRMPBF

Commit message: Schematic Almost Completed and PCB Tracing going on
Connections:
- net GND_A is gone; now on net GND: U1.4 (GND1)
- net NTC_3_IN is gone; now on net MOS_DRIVE_TRIGGER: R1.2, R24.1
- net 5V: now also U1.1 (VCC1)
- net GND: now also U1.8 (VEE2); no longer IC1.2 (K)
- net MOS_DRIVE_TRIGGER: now also U1.6 (OUT)
- net NTC_2_IN: now also IC1.2 (K)
- net IN+<-->PWM: now reaches U1.2 (IN+)
- net R20<->IN-: now reaches R20.2, U1.3 (IN-)
- net CLMP<-->R1: now reaches R1.1, U1.7 (CLAMP)
- net MCU/PWM_SIGNAL renamed MCU/GNDA
Other:
- moved on the sheet: IC1
Changed lines of the file:
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@@
+	)
+	(junction
+		(at 266.7 85.09)
+		(diameter 0)
+		(color 0 0 0 0)
 	)
 	(junction
@@
 	(wire
 		(pts
-			(xy 266.7 72.39) (xy 266.7 91.44)
+			(xy 266.7 72.39) (xy 266.7 85.09)
 		)
 		(stroke
@@
 	(wire
 		(pts
-			(xy 248.92 91.44) (xy 266.7 91.44)
-		)
-		(stroke
-			(width 0)
-			(type default)
-		)
-	)
-	(wire
-		(pts
 			(xy 77.47 105.41) (xy 77.47 106.68)
 		)
@@
 	(wire
 		(pts
+			(xy 191.77 85.09) (xy 194.31 87.63)
+		)
+		(stroke
+			(width 0)
+			(type default)
+		)
+	)
+	(wire
+		(pts
 			(xy 111.76 91.44) (xy 127 91.44)
 		)
@@
 	(wire
 		(pts
-			(xy 30.48 167.64) (xy 31.75 167.64)
-		)
-		(stroke
-			(width 0)
-			(type default)
-		)
-	)
-	(wire
-		(pts
 			(xy 29.21 19.05) (xy 31.75 19.05)
 		)
@@
 	(wire
 		(pts
-			(xy 158.75 39.37) (xy 158.75 85.09)
-		)
-		(stroke
-			(width 0)
-			(type default)
-		)
-	)
-	(wire
-		(pts
 			(xy 78.74 118.11) (xy 78.74 140.97)
 		)
@@
 	(wire
 		(pts
+			(xy 213.36 99.06) (xy 201.93 99.06)
+		)
+		(stroke
+			(width 0)
+			(type default)
+		)
+	)
+	(wire
+		(pts
 			(xy 45.72 128.27) (xy 73.66 128.27)
 		)
@@
 	(wire
 		(pts
-			(xy 158.75 39.37) (xy 160.02 39.37)
+			(xy 158.75 26.67) (xy 158.75 85.09)
 		)
 		(stroke
@@
 	(wire
 		(pts
-			(xy 213.36 95.25) (xy 213.36 99.06)
-		)
-		(stroke
-			(width 0)
-			(type default)
-		)
-	)
-	(wire
-		(pts
 			(xy 208.28 29.21) (xy 201.93 29.21)
 		)
@@
 	(wire
 		(pts
-			(xy 158.75 85.09) (xy 213.36 85.09)
-		)
-		(stroke
-			(width 0)
-			(type default)
-		)
-	)
-	(wire
-		(pts
 			(xy 44.45 127) (xy 41.91 127)
 		)
@@
 	(wire
 		(pts
-			(xy 213.36 99.06) (xy 201.93 99.06)
-		)
-		(stroke
-			(width 0)
-			(type default)
-		)
-	)
-	(wire
-		(pts
 			(xy 41.91 119.38) (xy 45.72 119.38)
 		)
@@
 	(wire
 		(pts
+			(xy 158.75 26.67) (xy 160.02 25.4)
+		)
+		(stroke
+			(width 0)
+			(type default)
+		)
+	)
+	(wire
+		(pts
 			(xy 208.28 38.1) (xy 208.28 44.45)
 		)
@@
 	(wire
 		(pts
-			(xy 157.48 25.4) (xy 160.02 25.4)
-		)
-		(stroke
-			(width 0)
-			(type default)
-		)
-	)
-	(wire
-		(pts
 			(xy 257.81 114.3) (xy 252.73 114.3)
 		)
@@
 	(wire
 		(pts
-			(xy 196.85 77.47) (xy 196.85 80.01)
+			(xy 158.75 85.09) (xy 191.77 85.09)
+		)
+		(stroke
+			(width 0)
+			(type default)
+		)
+	)
+	(wire
+		(pts
+			(xy 196.85 77.47) (xy 196.85 82.55)
 		)
 		(stroke
@@
 	(wire
 		(pts
+			(xy 31.75 167.64) (xy 30.48 167.64)
+		)
+		(stroke
+			(width 0)
+			(type default)
+		)
+	)
+	(wire
+		(pts
 			(xy 20.32 121.92) (xy 20.32 120.65)
 		)
@@
 	(wire
 		(pts
-			(xy 196.85 80.01) (xy 213.36 80.01)
+			(xy 196.85 82.55) (xy 213.36 82.55)
 		)
 		(stroke
@@
 	(wire
 		(pts
-			(xy 157.48 25.4) (xy 157.48 90.17)
+			(xy 157.48 39.37) (xy 157.48 90.17)
 		)
 		(stroke
@@
 	(wire
 		(pts
+			(xy 194.31 87.63) (xy 213.36 87.63)
+		)
+		(stroke
+			(width 0)
+			(type default)
+		)
+	)
+	(wire
+		(pts
+			(xy 266.7 85.09) (xy 266.7 90.17)
+		)
+		(stroke
+			(width 0)
+			(type default)
+		)
+	)
+	(wire
+		(pts
 			(xy 50.8 57.15) (xy 55.88 57.15)
 		)
@@
 	(wire
 		(pts
+			(xy 213.36 93.98) (xy 213.36 99.06)
+		)
+		(stroke
+			(width 0)
+			(type default)
+		)
+	)
+	(wire
+		(pts
 			(xy 167.64 123.19) (xy 167.64 125.73)
 		)
@@
 	(wire
 		(pts
+			(xy 248.92 90.17) (xy 266.7 90.17)
+		)
+		(stroke
+			(width 0)
+			(type default)
+		)
+	)
+	(wire
+		(pts
 			(xy 27.94 119.38) (xy 27.94 130.81)
 		)
@@
 		(pts
 			(xy 90.17 106.68) (xy 95.25 106.68)
+		)
+		(stroke
+			(width 0)
+			(type default)
+		)
+	)
+	(wire
+		(pts
+			(xy 157.48 39.37) (xy 160.02 39.37)
 		)
 		(stroke
@@
 		)
 	)
+	(label "DC-DC_CONV_GND"
+		(at 21.59 71.12 0)
+		(fields_autoplaced yes)
+		(effects
+			(font
+				(size 1.27 1.27)
+			)
+			(justify left bottom)
+		)
+	)
 	(label "GND_HIGH"
 		(at 252.73 96.52 0)
@@
 		)
 	)
+	(label "IN+<-->PWM"
+		(at 173.99 85.09 0)
+		(fields_autoplaced yes)
+		(effects
+			(font
+				(size 1.27 1.27)
+			)
+			(justify left bottom)
+		)
+	)
 	(label "Vin"
 		(at 29.21 19.05 180)
@@
 		)
 	)
-	(label "GND_A"
-		(at 204.47 85.09 0)
-		(fields_autoplaced yes)
-		(effects
-			(font
-				(size 1.27 1.27)
-			)
-			(justify left bottom)
-		)
-	)
 	(label "MOS_GND"
 		(at 27.94 128.27 0)
@@
 		)
 	)
+	(label "DC-DC_CONV_GND"
+		(at 31.75 167.64 0)
+		(fields_autoplaced yes)
+		(effects
+			(font
+				(size 1.27 1.27)
+			)
+			(justify left bottom)
+		)
+	)
 	(label "VCC3V3"
 		(at 226.06 21.59 0)
@@
 		)
 	)
-	(label "CLMP_MOS_DRIVE_TIGGER"
-		(at 256.54 91.44 0)
-		(fields_autoplaced yes)
-		(effects
-			(font
-				(size 1.27 1.27)
-			)
-			(justify left bottom)
-		)
-	)
 	(label "SW_PIN"
 		(at 259.08 21.59 0)
@@
 		)
 	)
+	(label "R20<->IN-"
+		(at 194.31 90.17 0)
+		(fields_autoplaced yes)
+		(effects
+			(font
+				(size 1.27 1.27)
+			)
+			(justify left bottom)
+		)
+	)
 	(label "mos_gate_input"
 		(at 39.37 114.3 0)
@@
 	(label "MOSFET_DRAIN_OUT"
 		(at 95.25 106.68 0)
+		(fields_autoplaced yes)
+		(effects
+			(font
+				(size 1.27 1.27)
+			)
+			(justify left bottom)
+		)
+	)
+	(label "CLMP<-->R1"
+		(at 250.19 85.09 0)
 		(fields_autoplaced yes)
 		(effects
@@
 	)
 	(global_label "NTC_3_OUT"
-		(shape input)
+		(shape output)
 		(at 231.14 128.27 0)
 		(fields_autoplaced yes)
